Commit message: change camera to correct location

File: urdf/udacity_bot.xacro (robot description, xacro)
@@ -185,5 +185,5 @@
   </link>
   <joint type="fixed" name="camera_joint">
-    <origin xyz="0.22 0 -0.0" rpy="0 0 0"/>
+    <origin xyz="0.23 0 0.18" rpy="0 0 0"/>
     <child link="camera"/>
     <parent link="chassis"/>

Commit message: environment is fully setup and ready for tuning

File: urdf/udacity_bot.xacro (robot description, xacro)
@@ -1,5 +1,5 @@
 <?xml version='1.0'?>
 <robot name="udacity_my_bot" xmlns:xacro="http://www.ros.org/wiki/xacro">
-  <!-- <xacro:include filename="$(find udacity_bot)/urdf/udacity_bot.gazebo"/> -->
+  <xacro:include filename="$(find udacity_my_robot)/urdf/udacity_bot.gazebo"/>
   <link name="robot_footprint"></link>
   <joint name="robot_footprint_joint" type="fixed">
@@ -211,5 +211,5 @@
     <visual name='hokuyo_visual'>
       <geometry>
-          <mesh filename="package://udacity_bot/meshes/hokuyo.dae"/>
+          <mesh filename="package://udacity_my_robot/meshes/hokuyo.dae"/>
       </geometry>
     </visual>

Commit message: robot can move and turn to simple goal

File: urdf/udacity_bot.xacro (robot description, xacro)
@@ -12,5 +12,5 @@
     <inertial>
       <mass value="15.0"/>
-      <origin xyz="0.0 0 0" rpy=" 0 0 0"/>
+      <origin xyz="0.0 0 0.15" rpy=" 0 0 0"/>
       <inertia
           ixx="0.1" ixy="0" ixz="0"
@@ -20,13 +20,13 @@
     </inertial>
     <collision name='collision'>
-      <origin xyz="0 0 0.12" rpy=" 0 0 0"/>
-      <geometry>
-        <box size=".4 .3 .15"/>
+      <origin xyz="0 0 0.15" rpy=" 0 0 0"/>
+      <geometry>
+        <box size=".4 .3 .12"/>
       </geometry>
     </collision>
     <visual name='chassis_visual'>
-      <origin xyz="0 0 0.12" rpy=" 0 0 0"/>
-      <geometry>
-        <box size=".4 .3 .15"/>
+      <origin xyz="0 0 0.15" rpy=" 0 0 0"/>
+      <geometry>
+        <box size=".4 .3 .12"/>
       </geometry>
     </visual>
@@ -35,5 +35,5 @@
   <link name='left_back_wheel'>
     <inertial>
-      <mass value="5.0"/>
+      <mass value="2.0"/>
       <origin xyz="0 0 0" rpy=" 0 1.5707 1.5707"/>
       <inertia
@@ -46,5 +46,5 @@
       <origin xyz="0 0 0" rpy=" 0 1.5707 1.5707"/>
       <geometry>
-        <cylinder length="0.07" radius="0.12"/>
+        <cylinder length="0.07" radius="0.10"/>
       </geometry>
     </collision>
@@ -52,5 +52,5 @@
       <origin xyz="0 0 0" rpy=" 0 1.5707 1.5707"/>
       <geometry>
-        <cylinder length="0.07" radius="0.12"/>
+        <cylinder length="0.07" radius="0.10"/>
       </geometry>
     </visual>
@@ -67,5 +67,5 @@
   <link name='left_front_wheel'>
     <inertial>
-      <mass value="5.0"/>
+      <mass value="2.0"/>
       <origin xyz="0 0 0" rpy=" 0 1.5707 1.5707"/>
       <inertia
@@ -78,5 +78,5 @@
       <origin xyz="0 0 0" rpy=" 0 1.5707 1.5707"/>
       <geometry>
-        <cylinder length="0.07" radius="0.12"/>
+        <cylinder length="0.07" radius="0.10"/>
       </geometry>
     </collision>
@@ -84,5 +84,5 @@
       <origin xyz="0 0 0" rpy=" 0 1.5707 1.5707"/>
       <geometry>
-        <cylinder length="0.07" radius="0.12"/>
+        <cylinder length="0.07" radius="0.10"/>
       </geometry>
     </visual>
@@ -99,5 +99,5 @@
   <link name='right_back_wheel'>
     <inertial>
-      <mass value="5.0"/>
+      <mass value="2.0"/>
       <origin xyz="0 0 0" rpy=" 0 1.5707 1.5707"/>
       <inertia
@@ -110,5 +110,5 @@
       <origin xyz="0 0 0" rpy=" 0 1.5707 1.5707"/>
       <geometry>
-        <cylinder length="0.07" radius="0.12"/>
+        <cylinder length="0.07" radius="0.10"/>
       </geometry>
     </collision>
@@ -116,5 +116,5 @@
       <origin xyz="0 0 0" rpy=" 0 1.5707 1.5707"/>
       <geometry>
-        <cylinder length="0.07" radius="0.12"/>
+        <cylinder length="0.07" radius="0.10"/>
       </geometry>
     </visual>
@@ -131,5 +131,5 @@
   <link name='right_front_wheel'>
     <inertial>
-      <mass value="5.0"/>
+      <mass value="2.0"/>
       <origin xyz="0 0 0" rpy=" 0 1.5707 1.5707"/>
       <inertia
@@ -142,5 +142,5 @@
       <origin xyz="0 0 0" rpy=" 0 1.5707 1.5707"/>
       <geometry>
-        <cylinder length="0.07" radius="0.12"/>
+        <cylinder length="0.07" radius="0.10"/>
       </geometry>
     </collision>
@@ -148,5 +148,5 @@
       <origin xyz="0 0 0" rpy=" 0 1.5707 1.5707"/>
       <geometry>
-        <cylinder length="0.07" radius="0.12"/>
+        <cylinder length="0.07" radius="0.10"/>
       </geometry>
     </visual>
@@ -216,5 +216,5 @@
   </link>
   <joint type="fixed" name="hokuyo_joint">
-    <origin xyz="0 0 0.4" rpy="0 0 0"/>
+    <origin xyz="0.1 0 0.4" rpy="0 0 0"/>
     <child link="hokuyo"/>
     <parent link="chassis"/>

Commit message: more improvement with high escape velocity

File: urdf/udacity_bot.xacro (robot description, xacro)
@@ -46,5 +46,5 @@
       <origin xyz="0 0 0" rpy=" 0 1.5707 1.5707"/>
       <geometry>
-        <cylinder length="0.07" radius="0.10"/>
+        <cylinder length="0.07" radius="0.08"/>
       </geometry>
     </collision>
@@ -52,5 +52,5 @@
       <origin xyz="0 0 0" rpy=" 0 1.5707 1.5707"/>
       <geometry>
-        <cylinder length="0.07" radius="0.10"/>
+        <cylinder length="0.07" radius="0.08"/>
       </geometry>
     </visual>
@@ -78,5 +78,5 @@
       <origin xyz="0 0 0" rpy=" 0 1.5707 1.5707"/>
       <geometry>
-        <cylinder length="0.07" radius="0.10"/>
+        <cylinder length="0.07" radius="0.08"/>
       </geometry>
     </collision>
@@ -84,5 +84,5 @@
       <origin xyz="0 0 0" rpy=" 0 1.5707 1.5707"/>
       <geometry>
-        <cylinder length="0.07" radius="0.10"/>
+        <cylinder length="0.07" radius="0.08"/>
       </geometry>
     </visual>
@@ -110,5 +110,5 @@
       <origin xyz="0 0 0" rpy=" 0 1.5707 1.5707"/>
       <geometry>
-        <cylinder length="0.07" radius="0.10"/>
+        <cylinder length="0.07" radius="0.08"/>
       </geometry>
     </collision>
@@ -116,5 +116,5 @@
       <origin xyz="0 0 0" rpy=" 0 1.5707 1.5707"/>
       <geometry>
-        <cylinder length="0.07" radius="0.10"/>
+        <cylinder length="0.07" radius="0.08"/>
       </geometry>
     </visual>
@@ -142,5 +142,5 @@
       <origin xyz="0 0 0" rpy=" 0 1.5707 1.5707"/>
       <geometry>
-        <cylinder length="0.07" radius="0.10"/>
+        <cylinder length="0.07" radius="0.08"/>
       </geometry>
     </collision>
@@ -148,5 +148,5 @@
       <origin xyz="0 0 0" rpy=" 0 1.5707 1.5707"/>
       <geometry>
-        <cylinder length="0.07" radius="0.10"/>
+        <cylinder length="0.07" radius="0.08"/>
       </geometry>
     </visual>

Commit message: very close to finish

File: urdf/udacity_bot.xacro (robot description, xacro)
@@ -206,5 +206,5 @@
       <origin xyz="0 0 0" rpy=" 0 0 0"/>
       <geometry>
-        <box size="0.1 0.1 0.4"/>
+        <box size="0.1 0.1 0.5"/>
       </geometry>
     </collision>
@@ -216,5 +216,5 @@
   </link>
   <joint type="fixed" name="hokuyo_joint">
-    <origin xyz="0.1 0 0.4" rpy="0 0 0"/>
+    <origin xyz="0 0 0.4" rpy="0 0 0"/>
     <child link="hokuyo"/>
     <parent link="chassis"/>

Commit message: final configuration and tuning

File: urdf/udacity_bot.xacro (robot description, xacro)
@@ -22,5 +22,5 @@
       <origin xyz="0 0 0.15" rpy=" 0 0 0"/>
       <geometry>
-        <box size=".4 .3 .12"/>
+        <box size=".35 .3 .11"/>
       </geometry>
     </collision>
@@ -28,5 +28,5 @@
       <origin xyz="0 0 0.15" rpy=" 0 0 0"/>
       <geometry>
-        <box size=".4 .3 .12"/>
+        <box size=".4 .3 .11"/>
       </geometry>
     </visual>
@@ -180,10 +180,10 @@
       <origin xyz="0 0 0" rpy=" 0 0 0"/>
       <geometry>
-        <box size="0.05 0.05 0.05"/>
+        <box size="0.02 0.02 0.02"/>
       </geometry>
     </visual>
   </link>
   <joint type="fixed" name="camera_joint">
-    <origin xyz="0.23 0 0.18" rpy="0 0 0"/>
+    <origin xyz="0.22 0 0.18" rpy="0 0 0"/>
     <child link="camera"/>
     <parent link="chassis"/>
@@ -216,5 +216,5 @@
   </link>
   <joint type="fixed" name="hokuyo_joint">
-    <origin xyz="0 0 0.4" rpy="0 0 0"/>
+    <origin xyz="-0.07 0 0.3" rpy="0 0 0"/>
     <child link="hokuyo"/>
     <parent link="chassis"/>

Commit message: ready for submission

File: urdf/udacity_bot.xacro (robot description, xacro)
@@ -67,5 +67,5 @@
   <link name='left_front_wheel'>
     <inertial>
-      <mass value="2.0"/>
+      <mass value="4.0"/>
       <origin xyz="0 0 0" rpy=" 0 1.5707 1.5707"/>
       <inertia
@@ -94,5 +94,5 @@
     <axis xyz="0 1 0" rpy="0 0 0"/>
     <limit effort="10000" velocity="1000"/>
-    <joint_properties damping="1.0" friction="1.0"/>
+    <joint_properties damping="1.0" friction="1.5"/>
   </joint>
 <!-- RIGHT BACK WHEEL -->
@@ -131,5 +131,5 @@
   <link name='right_front_wheel'>
     <inertial>
-      <mass value="2.0"/>
+      <mass value="4.0"/>
       <origin xyz="0 0 0" rpy=" 0 1.5707 1.5707"/>
       <inertia
@@ -158,5 +158,5 @@
     <axis xyz="0 1 0" rpy="0 0 0"/>
     <limit effort="10000" velocity="1000"/>
-    <joint_properties damping="1.0" friction="1.0"/>
+    <joint_properties damping="1.0" friction="1.5"/>
   </joint>
   <!-- CAMERA -->

Commit message: robot can go straigght now

File: urdf/udacity_bot.xacro (robot description, xacro)
@@ -28,5 +28,5 @@
       <origin xyz="0 0 0.15" rpy=" 0 0 0"/>
       <geometry>
-        <box size=".4 .3 .11"/>
+        <box size=".35 .3 .11"/>
       </geometry>
     </visual>
@@ -34,5 +34,5 @@
   <!-- LEFT BACK WHEEL -->
   <link name='left_back_wheel'>
-    <inertial>
+   <inertial>
       <mass value="2.0"/>
       <origin xyz="0 0 0" rpy=" 0 1.5707 1.5707"/>
@@ -94,5 +94,5 @@
     <axis xyz="0 1 0" rpy="0 0 0"/>
     <limit effort="10000" velocity="1000"/>
-    <joint_properties damping="1.0" friction="1.5"/>
+    <joint_properties damping="1.0" friction="1.0"/>
   </joint>
 <!-- RIGHT BACK WHEEL -->
@@ -158,5 +158,5 @@
     <axis xyz="0 1 0" rpy="0 0 0"/>
     <limit effort="10000" velocity="1000"/>
-    <joint_properties damping="1.0" friction="1.5"/>
+    <joint_properties damping="1.0" friction="1.0"/>
   </joint>
   <!-- CAMERA -->
@@ -216,5 +216,5 @@
   </link>
   <joint type="fixed" name="hokuyo_joint">
-    <origin xyz="-0.07 0 0.3" rpy="0 0 0"/>
+    <origin xyz="0.1 0 0.3" rpy="0 0 0"/>
     <child link="hokuyo"/>
     <parent link="chassis"/>
